File: supervisor_schematic/supervisor.kicad_pcb (KiCad board)
At the start: 2 copper layers, 45 parts, among them IC1 PCF8574DW, J1 J, J10 J, J11 J, J12 J, J13 J, J14 J, J15 J, J16 Conn_01x06_Female, J2 J, J3 J, J4 J, J5 J, J6 J, J7 J, J8 J, J9 J, SW1 SW_Push, SW2 SW_Push, SW3 SW_Push, U1 74HC14, U2 RFM9-LoRa-Radio

Commit message: started routing
Parts:
- removed C7: 100n, Capacitor_SMD:C_0805_2012Metric_Pad1.15x1.40mm_HandSolder
- removed IC1: PCF8574DW, Connector_PinHeader_2.54mm:PinHeader_1x04_P2.54mm_Vertical
- removed J10, J11, J12, J13, J14, J15, J3, J4, J5, J6, J7, J8, J9: J, Connector_PinHeader_2.54mm:PinHeader_1x01_P2.54mm_Vertical
- added J17: Conn_01x04_Female, Connector_PinHeader_2.54mm:PinHeader_1x04_P2.54mm_Vertical, F.Cu at (166.1, 92.7)
- J1: value J -> Conn_01x08; footprint Connector_PinHeader_2.54mm:PinHeader_1x01_P2.54mm_Vertical -> Connector_PinHeader_2.54mm:PinHeader_1x08_P2.54mm_Vertical
- J2: value J -> Conn_01x05; footprint Connector_PinHeader_2.54mm:PinHeader_1x01_P2.54mm_Vertical -> Connector_PinHeader_2.54mm:PinHeader_1x05_P2.54mm_Vertical
- moved U2 121.7 mm to (159.0, 116.3)
- moved C1 113.0 mm to (115.3, 82.3)
- moved R6 107.8 mm to (110.2, 81.3), turned to 270 degrees
- moved J2 102.3 mm to (173.7, 99.3)
- moved SW3 96.6 mm to (110.2, 85.9)
- moved J1 93.6 mm to (101.6, 96.0)
- moved CP4 93.3 mm to (128.0, 89.9), turned to 90 degrees
- moved D3 88.6 mm to (131.3, 78.2)
- moved Jack1 87.9 mm to (135.4, 73.4), turned to 270 degrees
- moved CP5 85.6 mm to (123.4, 89.9), turned to 90 degrees
- moved R9 84.0 mm to (137.4, 78.2)
- moved VR1 82.2 mm to (155.2, 73.2), turned to 270 degrees
- moved D2 70.7 mm to (131.3, 118.4), turned to 90 degrees
- moved D1 65.1 mm to (135.4, 118.4), turned to 90 degrees
- moved R8 63.9 mm to (131.3, 112.8), turned to 90 degrees
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Connections:
- J1 pad 1: IO27 -> GPIO36
- J2 pad 1: GPIO36 -> IO23
- U1 pad 2: Net-(U1-Pad2) -> IO25
- U1 pad 4: Net-(U1-Pad4) -> IO26
Routing:
- net +3V3: track 0.00 -> 216.4 mm, vias 0 -> 1
- net IO23: track 0.00 -> 49.9 mm, vias 0 -> 1
- net IO19: track 0.00 -> 26.5 mm, vias 0 -> 1
- net +5V: track 0.00 -> 26.0 mm, vias 0 -> 1
- net IO5: track 0.00 -> 25.3 mm, vias 0 -> 1
- net IO4: track 0.00 -> 24.8 mm, vias 0 -> 1
- net SCL: track 0.00 -> 24.3 mm, vias 0 -> 1
- net SDA: track 0.00 -> 23.1 mm, vias 0 -> 1
- net IO2: track 0.00 -> 22.2 mm, vias 0 -> 1
- net Net-(LS1-Pad1): track 0.00 -> 5.36 mm
Other:
- net class Default: clearance 0.2 -> 0.254; trace_width 0.25 -> 0.254; via_dia 0.8 -> 0.762; via_drill 0.4 -> 0.381
- rule pad_to_mask_clearance: 0.051 -> 0.0508
- rule solder_mask_min_width: 0.25 -> 0.1016
- rule trace_clearance: 0.2 -> 0.254
- rule trace_min: 0.2 -> 0.1524
- rule via_min_drill: 0.3 -> 0.254
- rule via_min_size: 0.4 -> 0.508

Commit message: supervisor done
Parts:
- added J3: Conn_01x02, Connector_PinHeader_2.54mm:PinHeader_1x02_P2.54mm_Vertical, F.Cu at (155.3, 136.8)
- added REF**: MountingHole_3.2mm_M3, MountingHole:MountingHole_3.2mm_M3, F.Cu at (110.5, 87.4)
- added REF**: MountingHole_3.2mm_M3, MountingHole:MountingHole_3.2mm_M3, F.Cu at (199.1, 137.4)
- added REF**: MountingHole_3.2mm_M3, MountingHole:MountingHole_3.2mm_M3, F.Cu at (111.0, 57.1)
- added REF**: MountingHole_3.2mm_M3, MountingHole:MountingHole_3.2mm_M3, F.Cu at (198.9, 57.4)
- moved C6 67.4 mm to (170.2, 114.0), turned to 270 degrees
- moved U2 15.0 mm to (174.0, 116.3)
- moved R5 14.0 mm to (152.4, 125.0)
- moved LS1 13.3 mm to (145.5, 135.0)
- moved SW1 9.43 mm to (120.7, 122.2)
- moved C2 9.43 mm to (116.3, 126.7)
- moved R1 9.43 mm to (116.3, 122.2)
- moved R2 9.43 mm to (131.8, 122.2)
- moved D1 9.26 mm to (142.2, 124.6)
- moved R7 9.26 mm to (142.2, 118.8), turned to 270 degrees
- moved D2 9.26 mm to (138.2, 124.6)
- moved R8 9.26 mm to (138.2, 119.0)
- moved ANT1 9.14 mm to (149.8, 95.8)
- moved C3 9.14 mm to (116.1, 136.7)
- moved CP4 9.14 mm to (137.2, 89.9)
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Routing:
- net IO13: track 0.00 -> 92.6 mm
- net RESET: track 0.00 -> 67.0 mm, vias 0 -> 3
- net IO0: track 0.00 -> 60.1 mm, vias 0 -> 1
- net IO18: track 0.00 -> 51.1 mm
- net Net-(C3-Pad1): track 0.00 -> 47.8 mm, vias 0 -> 1
- net CS: track 0.00 -> 47.7 mm, vias 0 -> 1
- net RX: track 0.00 -> 47.5 mm, vias 0 -> 3
- net SD3: track 0.00 -> 47.4 mm, vias 0 -> 1
- net SD2: track 0.00 -> 45.8 mm, vias 0 -> 1
- net TX: track 0.00 -> 44.4 mm, vias 0 -> 3
- net IO14: track 0.00 -> 43.8 mm, vias 0 -> 1
- net IO12: track 0.00 -> 41.9 mm, vias 0 -> 1
- net CLK: track 0.00 -> 39.4 mm, vias 0 -> 1
- net IO17: track 0.00 -> 35.7 mm, vias 0 -> 3
- net IO27: track 0.00 -> 35.5 mm, vias 0 -> 1
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- added copper zone on B.Cu, net GND
- added copper zone on F.Cu, net GND
Other:
- board outline added: 96.5 x 88.6 mm
- board text added: "1"
- board text added: "Purdue University ECE477 Team 19: Noggin Dev Shah Mooyeon Kim Ryan Domanski Akshaj Prasannakumar Rev: 3/3/22"

Commit message: v2 almost done
Parts:
- added Q1: BSS138, Package_TO_SOT_SMD:SOT-23, F.Cu at (191.0, 79.5)
- added Q2: BSS138, Package_TO_SOT_SMD:SOT-23, F.Cu at (191.0, 86.6)
- added R10: 10K, Resistor_SMD:R_0805_2012Metric_Pad1.15x1.40mm_HandSolder, F.Cu at (178.1, 79.5)
- added R11: 10K, Resistor_SMD:R_0805_2012Metric_Pad1.15x1.40mm_HandSolder, F.Cu at (179.6, 86.6)
- added R12: 10K, Resistor_SMD:R_0805_2012Metric_Pad1.15x1.40mm_HandSolder, F.Cu at (184.2, 79.8)
- added R13: 10K, Resistor_SMD:R_0805_2012Metric_Pad1.15x1.40mm_HandSolder, F.Cu at (194.8, 93.7)
- moved REF** 29.2 mm to (198.1, 108.2)
- moved J17 26.5 mm to (201.2, 87.1)
- moved CP4 1.02 mm to (136.1, 89.9)
Connections:
- J17 pad 3: SDA -> Net-(J17-Pad3)
- J17 pad 4: SCL -> Net-(J17-Pad4)
- J3 pad 1: SD0 -> SD2
- J3 pad 2: SD1 -> SD3
- U2 pad 6: SD2 -> SD0
- U2 pad 7: SD3 -> SD1
Routing:
- net +3V3: track 229.7 -> 279.3 mm
- net +5V: track 26.0 -> 73.8 mm, vias 1 -> 5
- net Net-(J17-Pad4): track 0.00 -> 29.1 mm, vias 0 -> 2
- net SCL: track 24.3 -> 45.3 mm, vias 1 -> 4
- net Net-(J17-Pad3): track 0.00 -> 20.2 mm
- net SD1: track 32.7 -> 51.7 mm, vias 2 -> 5
- net SDA: track 26.0 -> 40.8 mm, vias 1 -> 2
- net SD3: track 47.4 -> 33.0 mm
- net SD2: track 45.8 -> 32.5 mm
- net SD0: track 31.8 -> 36.7 mm, vias 2 -> 3
- net IO0: track 60.1 -> 61.7 mm
- net TX: track 44.4 -> 45.1 mm
- net GND: vias 3 -> 4

Commit message: ordered
Parts:
- removed J16: Conn_01x06_Female, Connector_PinHeader_2.54mm:PinHeader_1x06_P2.54mm_Vertical
- added C4: 1u, Capacitor_SMD:C_0805_2012Metric_Pad1.15x1.40mm_HandSolder, F.Cu at (198.4, 99.3)
- added J4: Conn_01x07_Female, Connector_PinHeader_2.54mm:PinHeader_1x07_P2.54mm_Vertical, F.Cu at (137.9, 56.4)
- added Q3: MMBT2222, Noggin:SOT95P240X114-3N, F.Cu at (137.4, 64.3)
- added Q4: MMBT2222, Noggin:SOT95P240X114-3N, F.Cu at (147.8, 64.1)
- added R14: 10K, Resistor_SMD:R_0805_2012Metric_Pad1.15x1.40mm_HandSolder, F.Cu at (199.6, 94.7)
- added R15: 10k, Resistor_SMD:R_0805_2012Metric_Pad1.15x1.40mm_HandSolder, F.Cu at (147.1, 69.6)
- added R16: 10k, Resistor_SMD:R_0805_2012Metric_Pad1.15x1.40mm_HandSolder, F.Cu at (139.2, 69.3)
- added SW4: SW_Push, Button_Switch_THT:SW_PUSH_6mm, F.Cu at (185.8, 97.3)
- D1, D2, D3: footprint Capacitor_SMD:C_0805_2012Metric_Pad1.15x1.40mm_HandSolder -> Noggin:0805_LED_Extended
- J1: value Conn_01x08 -> Conn_01x06; footprint Connector_PinHeader_2.54mm:PinHeader_1x08_P2.54mm_Vertical -> Connector_PinHeader_2.54mm:PinHeader_1x06_P2.54mm_Vertical
- J3: value Conn_01x02 -> Conn_01x04; footprint Connector_PinHeader_2.54mm:PinHeader_1x02_P2.54mm_Vertical -> Connector_PinHeader_2.54mm:PinHeader_1x04_P2.54mm_Vertical
- moved J2 66.7 mm to (108.7, 95.5)
- moved J1 62.2 mm to (155.4, 139.2), turned to 90 degrees
- moved REF** 50.2 mm to (106.4, 137.4)
- moved J3 44.8 mm to (180.6, 99.8), turned to 0 degrees
- moved R5 9.73 mm to (160.5, 119.6)
- moved REF** 3.56 mm to (107.4, 57.1)
- moved REF** 0.80 mm to (198.1, 57.7)
Connections:
- ANT1 pad 13: IO14 -> SCLK
- ANT1 pad 14: IO12 -> MISO
- ANT1 pad 16: IO13 -> MOSI
- ANT1 pad 19: CS -> CMD
- ANT1 pad 23: Net-(ANT1-Pad23) -> CS
- ANT1 pad 31: IO19 -> Net-(ANT1-Pad31)
- J1 pad 1: GPIO36 -> SD2
- J1 pad 2: GPIO39 -> SD3
- J1 pad 3: IO34 -> CMD
- J1 pad 4: IO35 -> CLK
- J1 pad 5: IO27 -> SD0
- J1 pad 6: IO14 -> SD1
- J2 pad 1: IO23 -> GPIO36
- J2 pad 2: IO19 -> GPIO39
- J2 pad 3: IO5 -> IO34
- J2 pad 4: IO4 -> IO35
- J2 pad 5: IO2 -> IO27
- J3 pad 1: SD2 -> IO23
- J3 pad 2: SD3 -> IO5
- R5 pad 2: Net-(ANT1-Pad23) -> Net-(ANT1-Pad31)
- U2 pad 5: CLK -> SCLK
- U2 pad 6: SD0 -> MISO
- U2 pad 7: SD1 -> MOSI
- VR1 pad 1: +5V -> +3V3
- VR1 pad 3: +3V3 -> +5V
Routing:
- net IO13: track 92.6 -> 0.00 mm
- net IO0: track 61.7 -> 148.6 mm, vias 1 -> 2
- net SCLK: track 0.00 -> 55.0 mm, vias 0 -> 1
- net MISO: track 0.00 -> 52.3 mm, vias 0 -> 2
- net MOSI: track 0.00 -> 44.2 mm, vias 0 -> 2
- net IO14: track 43.8 -> 0.00 mm, vias 1 -> 0
- net IO12: track 41.9 -> 0.00 mm, vias 1 -> 0
- net CMD: track 0.00 -> 35.9 mm, vias 0 -> 1
- net Net-(ANT1-Pad31): track 0.00 -> 31.1 mm, vias 0 -> 2
- net RTS: track 0.00 -> 20.0 mm
- net IO19: track 18.9 -> 0.00 mm, vias 1 -> 0
- net Net-(ANT1-Pad23): track 18.3 -> 0.00 mm
- net DTR: track 0.00 -> 17.2 mm
- net Net-(LS1-Pad1): track 13.4 -> 28.7 mm, vias 0 -> 2
- net SD1: track 51.7 -> 37.8 mm, vias 5 -> 0
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Other:
- board size 96.5 x 88.6 mm -> 102.4 x 88.6 mm
- board text added: "3v3"
- board text added: "DTR"
- board text added: "GND esp32"
- board text added: "IO0 esp32"
- board text added: "Lora 1"
- board text added: "Purdue University ECE477 Team 19: Noggin Dev Shah Mooyeon Kim Ryan Domanski Akshaj Prasannakumar Rev: 3/10/22"
- board text added: "u1 3v3"
- board text removed: "Purdue University ECE477 Team 19: Noggin Dev Shah Mooyeon Kim Ryan Domanski Akshaj Prasannakumar Rev: 3/3/22"
