File: wearer_schematic/wearer.sch (KiCad schematic (older format))
At the start: 50 parts, among them J1 Conn_01x02_Male, J2 Conn_01x06, J3 P4:5, J4 P7, J5 P14, J6 P16:18, J7 P23, Q1 AO3400A, SW1 SW_SPST, SW2 SW_Push, SW3 SW_Push, SW4 SW_Push, U1 MQ-9B, U2 SEN-11574, U3 74HC14, U4 ESP32-WROOM-32D, U5 LSM6DSLTR, U6 RFM9-LoRa-Radio

Commit message: progress
Parts:
- removed J2: Conn_01x06, Connector_PinHeader_2.54mm:PinHeader_1x06_P2.54mm_Vertical, symbol Connector_Generic:Conn_01x06
- removed J4: P7, Connector_PinHeader_2.54mm:PinHeader_1x01_P2.54mm_Vertical, symbol Connector:Conn_01x01_Male
- removed J5: P14, Connector_PinHeader_2.54mm:PinHeader_1x01_P2.54mm_Vertical, symbol Connector:Conn_01x01_Male
- removed J6: P16:18, Connector_PinHeader_2.54mm:PinHeader_1x03_P2.54mm_Vertical, symbol Connector:Conn_01x03_Male
- removed J7: P23, Connector_PinHeader_2.54mm:PinHeader_1x01_P2.54mm_Vertical, symbol Connector:Conn_01x01_Male
- added C11: 0.1uF, Capacitor_SMD:C_0805_2012Metric_Pad1.15x1.40mm_HandSolder, symbol Device:C_Small
- added C12, C13: 1uF, Capacitor_SMD:C_0805_2012Metric_Pad1.15x1.40mm_HandSolder, symbol Device:C_Small
- added H1, H2, H3, H4: MountingHole, MountingHole:MountingHole_3.2mm_M3, symbol Mechanical:MountingHole
- added J2: 01x07_Female, Connector_PinSocket_2.54mm:PinSocket_1x07_P2.54mm_Vertical, symbol Connector:Conn_01x07_Female
- added J4: Conn_01x02_Female, Connector_PinSocket_2.54mm:PinSocket_1x02_P2.54mm_Vertical, symbol Connector:Conn_01x02_Female
- added J5: P17:18, Connector_PinHeader_2.54mm:PinHeader_1x02_P2.54mm_Vertical, symbol Connector:Conn_01x02_Male
- added Q2, Q3: MMBT2222, noggin:MMBT2222, symbol Transistor_BJT:MMBT3904
- added R18, R19, R20: 10k, Resistor_SMD:R_0805_2012Metric_Pad1.15x1.40mm_HandSolder, symbol Device:R
- added SW5: SW_Push, Button_Switch_THT:SW_PUSH_6mm, symbol Switch:SW_Push
- C9: footprint Capacitor_SMD:C_0805_2012Metric_Pad1.15x1.40mm_HandSolder -> Capacitor_THT:CP_Radial_D6.3mm_P2.50mm; symbol Device:C_Small -> Device:CP1_Small
- J1: footprint Connector_PinHeader_2.54mm:PinHeader_1x02_P2.54mm_Horizontal -> Connector_PinHeader_2.54mm:PinHeader_1x02_P2.54mm_Vertical
Connections:
- net P14 is gone; now on net SPI_MISO: U4.14 (IO12)
- net P16 is gone; now on net SPI_MOSI: U4.16 (IO13)
- net P23 is gone; now on net SPI_CS: U4.23 (IO15)
- net P7 is gone; now on net GPIO35_LED: U4.7 (IO35)
- net +3V3: now also J4.1 (Pin_1), R18.2
- net ADC1_CH6_BAT: now also C11.2
- net EN: now also Q3.3 (C)
- net GND: now also C9.2, C11.1, C12.1, C13.2, J2.6 (Pin_6), J4.2 (Pin_2), SW5.1; no longer C9.1
- net GPIO0: now also C13.1, Q2.3 (C), R18.1, SW5.2
- net P17: now also J5.1 (Pin_1)
- net P18: now also J5.2 (Pin_2)
- net SPI_CS: no longer U4.19 (CMD)
- net SPI_MISO: no longer U4.21 (SD0)
- net SPI_MOSI: no longer U4.22 (SD1)
- net SPI_SCK: now also U4.13 (IO14); no longer U4.20 (CLK)
- net at R2.2, SW1.2 (B), VR2.3 (VIN): now also C9.1, C12.2; no longer C9.2
- net GPIO14_LED renamed GPIO35_LED
- net GPIO35_LED: no longer U4.13 (IO14)
- net RX renamed ESP_RX
- net ESP_RX: now also J2.3 (Pin_3)
- net TX renamed ESP_TX
- net ESP_TX: now also J2.2 (Pin_2)
- new net: Q2.1 (B), R19.2
- new net: Q3.1 (B), R20.2
- new net DTR: J2.1 (Pin_1), Q2.2 (E), R20.1
- new net RTS: J2.7 (Pin_7), Q3.2 (E), R19.1
Other:
- note added: "EN and GPIO0 Programming"
- note added: "GPIO0"
- moved on the sheet: C1, J1, J3, R2, R3, R8, SW1, SW4

Commit message: before order
Parts:
- D1, D2: footprint LED_SMD:LED_0805_2012Metric_Pad1.15x1.40mm_HandSolder -> noggin:0805_LED_Extended
Changed lines of the file:
@@
-$EndComp
-$Comp
-L Noggin:U1V10F5 VR1
-U 1 1 621A437E
-P 1050 3900
-F 0 "VR1" V 1350 4000 50  0000 C CNN
-F 1 "U1V10F5" V 1250 3900 50  0000 C CNN
-F 2 "noggin:U1V10F5-VR" H 1050 3650 50  0001 C CNN
-F 3 "" H 1050 3650 50  0001 C CNN
-	1    1050 3900
-	0    -1   -1   0
 $EndComp
 $Comp
@@
 F 0 "D1" H 8593 3666 50  0000 C CNN
 F 1 "LED" H 8593 3575 50  0000 C CNN
-F 2 "LED_SMD:LED_0805_2012Metric_Pad1.15x1.40mm_HandSolder" H 8600 3450 50  0001 C CNN
+F 2 "noggin:0805_LED_Extended" H 8600 3450 50  0001 C CNN
 F 3 "~" H 8600 3450 50  0001 C CNN
 	1    8600 3450
@@
 F 0 "D2" H 8993 3666 50  0000 C CNN
 F 1 "LED" H 8993 3575 50  0000 C CNN
-F 2 "LED_SMD:LED_0805_2012Metric_Pad1.15x1.40mm_HandSolder" H 9000 3450 50  0001 C CNN
+F 2 "noggin:0805_LED_Extended" H 9000 3450 50  0001 C CNN
 F 3 "~" H 9000 3450 50  0001 C CNN
 	1    9000 3450
@@
 	1    0    0    -1
 $EndComp
+$Comp
+L Noggin:U1V10F5 VR1
+U 1 1 621A437E
+P 1050 3900
+F 0 "VR1" V 1350 4000 50  0000 C CNN
+F 1 "U1V10F5" V 1250 3900 50  0000 C CNN
+F 2 "noggin:U1V10F5-VR" H 1050 3650 50  0001 C CNN
+F 3 "" H 1050 3650 50  0001 C CNN
+	1    1050 3900
+	0    -1   -1   0
+$EndComp
 $EndSCHEMATC
