File: wearer_schematic/wearer.kicad_pcb (KiCad board)
At the start: 2 copper layers, 92.7 x 69.8 mm, 49 parts, among them J1 Conn_01x02_Male, J2 Conn_01x06, J3 P4:5, J4 P7, J5 P14, J6 P16:18, J7 P23, Q1 AO3400A, SW1 SW_SPST, SW2 SW_Push, SW3 SW_Push, SW4 SW_Push, U1 MQ-9B, U2 SEN-11574, U3 74HC14, U4 ESP32-WROOM-32D, U5 LSM6DSLTR, U6 RFM9-LoRa-Radio

Commit message: ground planes
Routing:
- net GND: track 0.00 -> 4.44 mm, vias 0 -> 4
- net Net-(C6-Pad1): track 36.9 -> 38.7 mm
- net SDO: track 15.3 -> 14.3 mm
- added copper zone on B.Cu, net GND
- added copper zone on F.Cu, net GND
Changed lines of the file:
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@@
     (thickness 1.6)
     (drawings 18)
-    (tracks 377)
+    (tracks 390)
     (zones 0)
     (modules 49)
@@
   )
   (setup
-    (last_trace_width 0.254)
+    (last_trace_width 0.4064)
     (user_trace_width 0.2032)
     (user_trace_width 0.254)
@@
     (descr "14-lead though-hole mounted DIP package, row spacing 7.62 mm (300 mils)")
     (tags "THT DIP DIL PDIP 2.54mm 7.62mm 300mil")
-    (fp_text reference U3 (at 3.81 -2.33) (layer F.SilkS)
+    (fp_text reference U3 (at 5.334 17.653) (layer F.SilkS)
       (effects (font (size 1 1) (thickness 0.15)))
     )
@@
   (gr_line (start 219.71 127) (end 219.71 57.15) (layer Edge.Cuts) (width 0.05))
   (gr_line (start 127 127) (end 219.71 127) (layer Edge.Cuts) (width 0.05))
-  (gr_text 23 (at 194.056 131.826 90) (layer F.SilkS)
+  (gr_text 23 (at 191.262 111.252) (layer F.SilkS)
     (effects (font (size 1.016 1.016) (thickness 0.2032)))
   )
@@
     (effects (font (size 1.27 1.27) (thickness 0.2286)))
   )
-  (gr_text 1* (at 177.8 107.95) (layer F.SilkS)
+  (gr_text 1* (at 177.8 106.68) (layer F.SilkS)
     (effects (font (size 1.5 1.5) (thickness 0.3)))
   )
@@
     (effects (font (size 1.5 1.5) (thickness 0.3)))
   )
+  (via (at 187.706 84.836) (size 0.6858) (drill 0.3302) (layers F.Cu B.Cu) (net 1))
+  (segment (start 197.354063 80.6577) (end 196.853937 80.6577) (width 0.2032) (layer F.Cu) (net 1))
+  (segment (start 196.853937 80.6577) (end 196.853937 81.530063) (width 0.2032) (layer F.Cu) (net 1))
+  (segment (start 196.853937 81.530063) (end 195.834 82.55) (width 0.2032) (layer F.Cu) (net 1))
+  (segment (start 195.834 82.55) (end 195.834 82.55) (width 0.2032) (layer F.Cu) (net 1))
+  (via (at 195.834 82.55) (size 0.6858) (drill 0.3302) (layers F.Cu B.Cu) (net 1))
+  (segment (start 198.0184 79.502) (end 198.0184 79.001874) (width 0.2032) (layer F.Cu) (net 1))
+  (via (at 199.136 78.994) (size 0.6858) (drill 0.3302) (layers F.Cu B.Cu) (net 1))
+  (segment (start 198.0184 79.001874) (end 199.128126 79.001874) (width 0.2032) (layer F.Cu) (net 1))
+  (segment (start 199.128126 79.001874) (end 199.136 78.994) (width 0.2032) (layer F.Cu) (net 1))
+  (via (at 174.244 80.264) (size 0.6858) (drill 0.3302) (layers F.Cu B.Cu) (net 1))
   (segment (start 170.185787 69.27) (end 165.1 69.27) (width 0.254) (layer F.Cu) (net 2))
   (segment (start 171.6 69.27) (end 170.185787 69.27) (width 0.254) (layer F.Cu) (net 2))
@@
   (segment (start 194.31 72.009) (end 193.421 71.12) (width 0.2032) (layer F.Cu) (net 6))
   (segment (start 193.421 71.12) (end 190.754 71.12) (width 0.2032) (layer F.Cu) (net 6))
-  (segment (start 198.0184 80.002126) (end 198.536816 80.002126) (width 0.2032) (layer F.Cu) (net 6))
   (via (at 199.644 77.724) (size 0.6858) (drill 0.3302) (layers F.Cu B.Cu) (net 6))
-  (segment (start 199.644 78.894942) (end 199.644 77.724) (width 0.2032) (layer F.Cu) (net 6))
-  (segment (start 198.536816 80.002126) (end 199.644 78.894942) (width 0.2032) (layer F.Cu) (net 6))
   (via (at 195.58 73.152) (size 0.6858) (drill 0.3302) (layers F.Cu B.Cu) (net 6))
   (segment (start 199.644 77.724) (end 199.644 77.239067) (width 0.2032) (layer B.Cu) (net 6))
@@
   (segment (start 194.31 78.486) (end 194.31 73.152) (width 0.2032) (layer F.Cu) (net 6))
   (segment (start 194.31 73.152) (end 194.31 72.009) (width 0.2032) (layer F.Cu) (net 6))
+  (segment (start 198.0184 80.002126) (end 200.144126 80.002126) (width 0.2032) (layer F.Cu) (net 6))
+  (segment (start 200.144126 80.002126) (end 200.644252 79.502) (width 0.2032) (layer F.Cu) (net 6))
+  (segment (start 200.644252 78.724252) (end 199.644 77.724) (width 0.2032) (layer F.Cu) (net 6))
+  (segment (start 200.644252 79.502) (end 200.644252 78.724252) (width 0.2032) (layer F.Cu) (net 6))
   (segment (start 147.32 93.735) (end 152.4 93.735) (width 0.254) (layer F.Cu) (net 7))
   (segment (start 152.4 85.335) (end 147.32 85.335) (width 0.254) (layer F.Cu) (net 8))
@@
   (segment (start 181.864 114.935) (end 180.34 114.935) (width 0.254) (layer B.Cu) (net 41))
   (segment (start 183.388 113.411) (end 181.864 114.935) (width 0.254) (layer B.Cu) (net 41))
-  (via (at 196.342 81.915) (size 0.6858) (drill 0.3302) (layers F.Cu B.Cu) (net 44))
-  (segment (start 196.353811 80.6577) (end 196.353811 81.903189) (width 0.2032) (layer F.Cu) (net 44))
-  (segment (start 196.353811 81.903189) (end 196.342 81.915) (width 0.2032) (layer F.Cu) (net 44))
   (segment (start 186.182 81.534) (end 182.686002 81.534) (width 0.2032) (layer F.Cu) (net 44))
   (segment (start 182.686002 81.534) (end 182.520001 81.700001) (width 0.2032) (layer F.Cu) (net 44))
-  (segment (start 195.961 81.534) (end 196.342 81.915) (width 0.2032) (layer B.Cu) (net 44))
   (via (at 186.182 81.534) (size 0.6858) (drill 0.3302) (layers F.Cu B.Cu) (net 44))
-  (segment (start 186.182 81.534) (end 195.961 81.534) (width 0.2032) (layer B.Cu) (net 44))
+  (segment (start 195.972811 80.6577) (end 195.350511 81.28) (width 0.2032) (layer F.Cu) (net 44))
+  (segment (start 196.353811 80.6577) (end 195.972811 80.6577) (width 0.2032) (layer F.Cu) (net 44))
+  (via (at 194.564 81.28) (size 0.6858) (drill 0.3302) (layers F.Cu B.Cu) (net 44))
+  (segment (start 195.350511 81.28) (end 194.564 81.28) (width 0.2032) (layer F.Cu) (net 44))
+  (segment (start 186.436 81.28) (end 186.182 81.534) (width 0.2032) (layer B.Cu) (net 44))
+  (segment (start 194.564 81.28) (end 186.436 81.28) (width 0.2032) (layer B.Cu) (net 44))
   (via (at 197.104 86.741) (size 0.6858) (drill 0.3302) (layers F.Cu B.Cu) (net 46))
   (segment (start 182.520001 89.320001) (end 194.524999 89.320001) (width 0.2032) (layer F.Cu) (net 46))
@@
   (segment (start 147.311 71.111) (end 147.32 71.12) (width 0.6096) (layer F.Cu) (net 64))
   (segment (start 142.24 71.111) (end 147.311 71.111) (width 0.6096) (layer F.Cu) (net 64))
+  (zone (net 1) (net_name GND) (layer F.Cu) (hatch edge 0.508)
+    (connect_pads (clearance 0.508))
+    (min_thickness 0.254)
+    (fill yes (arc_segments 32) (thermal_gap 0.508) (thermal_bridge_width 0.508))
+    (polygon
+      (pts
+        (xy 219.964 127.254) (xy 126.746 127.254) (xy 126.746 56.896) (xy 219.964 56.896)
+      )
+    )
+  )
+  (zone (net 1) (net_name GND) (layer B.Cu) (hatch edge 0.508)
+    (connect_pads (clearance 0.508))
+    (min_thickness 0.254)
+    (fill yes (arc_segments 32) (thermal_gap 0.508) (thermal_bridge_width 0.508))
+    (polygon
+      (pts
+        (xy 219.964 127.254) (xy 126.746 127.254) (xy 126.746 56.896) (xy 219.964 56.896)
+      )
+    )
+  )
 )

Commit message: pcb
Parts:
- added REF**: 3.2mm, MountingHole:MountingHole_3.2mm_M3, F.Cu at (215.6, 117.1)
- added REF**: 3.2mm, MountingHole:MountingHole_3.2mm_M3, F.Cu at (215.9, 61.0)
- added REF**: 3.2mm, MountingHole:MountingHole_3.2mm_M3, F.Cu at (131.4, 61.6)
- added REF**: 3.2mm, MountingHole:MountingHole_3.2mm_M3, F.Cu at (131.4, 122.6)
- moved LS1 4.49 mm to (211.5, 70.5)
- moved J1 2.54 mm to (129.5, 74.9)
- moved R15 2.29 mm to (203.2, 65.4)
Routing:
- net Net-(J1-Pad1): track 7.45 -> 9.99 mm
- net SDA: vias 0 -> 1
- net GPIO18_ACC: vias 0 -> 1
- net EN: vias 1 -> 2
Other:
- board text added: "Purdue University ECE477 Team 19: Noggin Dev Shah Mooyeon Kim Ryan Domanski Akshaj Prasannakumar Rev: 3/3/22"
- board text added: "T10"
- board text added: "T11"
- board text added: "T12"
- board text added: "T13"
- board text added: "T19"
- board text added: "T20"
- board text added: "T21"
- board text added: "T22"
- board text added: "T24"
- board text added: "T26"
- board text added: "T27"
- board text added: "T28"
- board text added: "T29"
- board text added: "T3"
- board text added: "T30"
- board text added: "T31"
- board text added: "T33"
- board text added: "T34"
- board text added: "T35"
- board text added: "T36"
- board text added: "T37"
- board text added: "T6"
- board text added: "T7"
- board text added: "T8"
- board text added: "T9"

Commit message: pcb cleanup
Parts:
- moved REF** 0.72 mm to (215.4, 61.5)
- moved REF** 0.25 mm to (215.4, 117.1)
- moved REF** 0.18 mm to (131.3, 61.5)
- moved REF** 0.18 mm to (131.3, 122.7)
Changed lines of the file:
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@@
   )
   (setup
-    (last_trace_width 0.6096)
+    (last_trace_width 0.2032)
     (user_trace_width 0.2032)
     (user_trace_width 0.254)
@@
   )
   (module MountingHole:MountingHole_3.2mm_M3 (layer F.Cu)
-    (at 215.646 117.094)
+    (at 215.392 117.094)
     (descr "Mounting Hole 3.2mm, no annular, M3")
     (tags "mounting hole 3.2mm no annular m3")
@@
   )
   (module MountingHole:MountingHole_3.2mm_M3 (layer F.Cu)
-    (at 215.9 60.96)
+    (at 215.392 61.468)
     (descr "Mounting Hole 3.2mm, no annular, M3")
     (tags "mounting hole 3.2mm no annular m3")
@@
   )
   (module MountingHole:MountingHole_3.2mm_M3 (layer F.Cu)
-    (at 131.445 61.595)
+    (at 131.318 61.468)
     (descr "Mounting Hole 3.2mm, no annular, M3")
     (tags "mounting hole 3.2mm no annular m3")
@@
   )
   (module MountingHole:MountingHole_3.2mm_M3 (layer F.Cu)
-    (at 131.445 122.555)
-    (descr "Mounting Hole 3.2mm, no annular, M3")
-    (tags "mounting hole 3.2mm no annular m3")
+    (at 131.318 122.682)
+    (descr "Mounting Hole 3.2mm, no annular, M3")
+    (tags "mounting hole 3.2mm no annular m3")

Commit message: update pcb
Parts:
- added C10: 0.1uF, Capacitor_SMD:C_0805_2012Metric_Pad1.15x1.40mm_HandSolder, F.Cu at (149.2, 96.3)
- moved C6 10.6 mm to (200.9, 81.3), turned to 270 degrees
- moved SW4 5.48 mm to (166.1, 59.4)
- moved C4 3.74 mm to (158.6, 80.6)
- moved R8 2.62 mm to (181.4, 66.2), turned to 270 degrees
- moved C5 1.42 mm to (161.3, 80.6)
- moved R15 1.40 mm to (204.6, 65.3), turned to 270 degrees
- moved C1 0.92 mm to (178.1, 63.1)
Connections:
- C6 pad 1: Net-(C6-Pad1) -> +3V3
- R16 pad 1: Net-(C6-Pad1) -> +3V3
- R17 pad 1: Net-(C6-Pad1) -> +3V3
- U5 pad 12: Net-(C6-Pad1) -> +3V3
- U5 pad 5: Net-(C6-Pad1) -> +3V3
Routing:
- net +3V3: track 243.8 -> 318.0 mm, vias 0 -> 3
- net Net-(C6-Pad1): track 38.7 -> 0.00 mm, vias 2 -> 0
- net GPIO0: track 49.8 -> 70.5 mm, vias 1 -> 5
- net GPIO26_BUZZ: track 55.6 -> 72.0 mm
- net EN: track 43.4 -> 47.4 mm, vias 2 -> 1
- net GPIO16_LORA: track 14.5 -> 17.9 mm, vias 0 -> 1
- net GND: track 4.44 -> 7.11 mm, vias 4 -> 7
- net ADC1_CH5_GAS: track 23.7 -> 26.1 mm
- net SPI_CS: track 31.3 -> 33.3 mm, vias 1 -> 2
- net P5: track 33.4 -> 31.6 mm
- net SDA: track 23.5 -> 21.9 mm
- net Net-(Q1-Pad3): track 14.3 -> 15.6 mm
- net P7: track 34.4 -> 35.0 mm
- net P4: track 29.4 -> 29.5 mm, vias 2 -> 1
- net GPIO4_LORA: vias 1 -> 0
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Other:
- net class Default: clearance 0.2032 -> 0.1524
- rule trace_clearance: 0.2032 -> 0.1524
- board text added: "16 17 18"
- board text removed: "18 17 16"

Commit message: update pcb
Parts:
- moved C8 2.96 mm to (202.2, 77.2), turned to 0 degrees
- moved C6 1.42 mm to (202.2, 80.6), turned to 0 degrees
Routing:
- net +3V3: track 318.0 -> 309.4 mm
