File: wearer_schematic/wearer.kicad_pcb (KiCad board)
At the start: 2 copper layers, 92.7 x 69.8 mm, 54 parts, among them J1 Conn_01x02_Male, J2 Conn_01x06, J3 P4:5, J4 P7, J5 P14, J6 P16:18, J7 P23, Q1 AO3400A, SW1 SW_SPST, SW2 SW_Push, SW3 SW_Push, SW4 SW_Push, U1 MQ-9B, U2 SEN-11574, U3 74HC14, U4 ESP32-WROOM-32D, U5 LSM6DSLTR, U6 RFM9-LoRa-Radio

Commit message: progress
Parts:
- removed J6: P16:18, Connector_PinHeader_2.54mm:PinHeader_1x03_P2.54mm_Vertical
- removed J7: P23, Connector_PinHeader_2.54mm:PinHeader_1x01_P2.54mm_Vertical
- removed REF** (x4): 3.2mm, MountingHole:MountingHole_3.2mm_M3
- added C11: 0.1uF, Capacitor_SMD:C_0805_2012Metric_Pad1.15x1.40mm_HandSolder, F.Cu at (144.5, 60.2)
- added C12: 1uF, Capacitor_SMD:C_0805_2012Metric_Pad1.15x1.40mm_HandSolder, F.Cu at (143.3, 72.1)
- added C13: 1uF, Capacitor_SMD:C_0805_2012Metric_Pad1.15x1.40mm_HandSolder, F.Cu at (177.8, 59.9)
- added H1: MountingHole, MountingHole:MountingHole_3.2mm_M3, F.Cu at (130.8, 61.0)
- added H2: MountingHole, MountingHole:MountingHole_3.2mm_M3, F.Cu at (130.8, 123.2)
- added H3: MountingHole, MountingHole:MountingHole_3.2mm_M3, F.Cu at (215.9, 61.0)
- added H4: MountingHole, MountingHole:MountingHole_3.2mm_M3, F.Cu at (215.9, 116.8)
- added Q2: MMBT2222, noggin:MMBT2222, F.Cu at (202.4, 68.8)
- added Q3: MMBT2222, noggin:MMBT2222, F.Cu at (212.9, 68.8)
- added R18: 10k, Resistor_SMD:R_0805_2012Metric_Pad1.15x1.40mm_HandSolder, F.Cu at (177.8, 64.3)
- added R19: 10k, Resistor_SMD:R_0805_2012Metric_Pad1.15x1.40mm_HandSolder, F.Cu at (207.8, 67.8)
- added R20: 10k, Resistor_SMD:R_0805_2012Metric_Pad1.15x1.40mm_HandSolder, F.Cu at (207.8, 64.5)
- added SW5: SW_Push, Button_Switch_THT:SW_PUSH_6mm, F.Cu at (181.9, 58.9)
- C9: footprint Capacitor_SMD:C_0805_2012Metric_Pad1.15x1.40mm_HandSolder -> Capacitor_THT:CP_Radial_D6.3mm_P2.50mm
- J2: value Conn_01x06 -> 01x07_Female; footprint Connector_PinHeader_2.54mm:PinHeader_1x06_P2.54mm_Vertical -> Connector_PinSocket_2.54mm:PinSocket_1x07_P2.54mm_Vertical
- J4: value P7 -> Conn_01x02_Female; footprint Connector_PinHeader_2.54mm:PinHeader_1x01_P2.54mm_Vertical -> Connector_PinSocket_2.54mm:PinSocket_1x02_P2.54mm_Vertical
- J5: value P14 -> P17:18; footprint Connector_PinHeader_2.54mm:PinHeader_1x01_P2.54mm_Vertical -> Connector_PinHeader_2.54mm:PinHeader_1x02_P2.54mm_Vertical
- moved J4 29.2 mm to (142.0, 85.3), turned to 0 degrees
- moved R15 22.8 mm to (203.4, 88.0), turned to 180 degrees
- moved LS1 13.7 mm to (212.4, 84.2), turned to 180 degrees
- moved R8 9.09 mm to (172.5, 64.3)
- moved D1 7.44 mm to (148.3, 85.3), turned to 90 degrees
- moved R13 7.44 mm to (153.4, 85.3), turned to 270 degrees
- moved C1 6.49 mm to (172.5, 59.8), turned to 90 degrees
- moved VR1 6.27 mm to (131.3, 83.6)
- moved J2 5.30 mm to (194.3, 61.2), turned to 90 degrees
- moved J3 5.21 mm to (156.8, 59.3)
- moved D2 4.81 mm to (148.3, 91.1)
- moved R14 4.81 mm to (153.4, 91.1)
- moved C9 4.58 mm to (137.7, 72.4), turned to 270 degrees
- moved SW4 3.94 mm to (162.2, 58.9)
- moved J5 1.83 mm to (166.1, 104.4), turned to 90 degrees
Connections:
- net RX renamed ESP_RX
- net TX renamed ESP_TX
- C9 pad 1: GND -> Net-(C12-Pad2)
- C9 pad 2: Net-(C9-Pad2) -> GND
- J2 pad 1: GND -> DTR
- J2 pad 4: +3V3 -> Net-(J2-Pad4)
- J2 pad 5: EN -> Net-(J2-Pad5)
- J2 pad 6: GPIO0 -> GND
- J4 pad 1: P7 -> +3V3
- J5 pad 1: P14 -> P17
- R13 pad 2: GPIO14_LED -> GPIO35_LED
- R2 pad 2: Net-(C9-Pad2) -> Net-(C12-Pad2)
- SW1 pad 2: Net-(C9-Pad2) -> Net-(C12-Pad2)
- U1 pad 2: +5V -> Net-(Q1-Pad3)
- U1 pad 5: Net-(Q1-Pad3) -> +5V
- U4 pad 13: GPIO14_LED -> SPI_SCK
- U4 pad 14: P14 -> SPI_MISO
- U4 pad 16: P16 -> SPI_MOSI
- U4 pad 19: SPI_CS -> Net-(U4-Pad19)
- U4 pad 20: SPI_SCK -> Net-(U4-Pad20)
- U4 pad 21: SPI_MISO -> Net-(U4-Pad21)
- U4 pad 22: SPI_MOSI -> Net-(U4-Pad22)
- U4 pad 23: P23 -> SPI_CS
- U4 pad 7: P7 -> GPIO35_LED
- VR2 pad 3: Net-(C9-Pad2) -> Net-(C12-Pad2)
Routing:
- net GPIO0: track 70.5 -> 12.9 mm, vias 5 -> 0
- net P7: track 35.0 -> 0.00 mm, vias 1 -> 0
- net GPIO26_BUZZ: track 72.0 -> 44.9 mm
- net P23: track 26.9 -> 0.00 mm, vias 2 -> 0
- net ESP_RX: track 28.1 -> 2.92 mm
- net ESP_TX: track 28.0 -> 2.92 mm
- net Net-(C12-Pad2): track 0.00 -> 21.8 mm
- net DTR: track 0.00 -> 18.9 mm, vias 0 -> 1
- net SPI_SCK: track 36.8 -> 54.2 mm, vias 1 -> 0
- net SPI_MISO: track 32.2 -> 48.8 mm, vias 1 -> 0
- net Net-(C9-Pad2): track 16.2 -> 0.00 mm
- net GPIO14_LED: track 15.1 -> 0.00 mm, vias 2 -> 0
- net GPIO35_LED: track 0.00 -> 13.8 mm, vias 0 -> 2
- net EN: track 47.4 -> 36.1 mm
- net RTS: track 0.00 -> 9.90 mm, vias 0 -> 1
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Other:
- board text added: "17 18"
- board text added: "3V3"
- board text added: "T14"
- board text added: "T16"
- board text added: "T23"
- board text removed: "*GND"
- board text removed: "14"
- board text removed: "16 17 18"
- board text removed: "23"
- board text removed: "7"
- board text removed: "IO0"
- board text removed: "T19"
- board text removed: "T20"
- board text removed: "T21"
- board text removed: "T22"

Commit message: pcb
Parts:
- moved H2 6.35 mm to (130.8, 116.8)
- moved Q2 1.70 mm to (201.7, 67.3), turned to 180 degrees
Routing:
- net GPIO0: track 12.9 -> 80.6 mm, vias 0 -> 2
- net EN: track 36.1 -> 84.3 mm, vias 1 -> 2
- net ESP_RX: track 2.92 -> 45.1 mm
- net ESP_TX: track 2.92 -> 44.2 mm
- net Net-(Q3-Pad1): track 7.86 -> 6.82 mm
- net Net-(Q2-Pad1): track 4.98 -> 4.05 mm
- net GND: vias 7 -> 8
Other:
- board text added: "DTR.ETX.ERX"
- board text added: "GND.RTS"
- board text added: "x x"

Commit message: before order
Parts:
- D1, D2: footprint LED_SMD:LED_0805_2012Metric_Pad1.15x1.40mm_HandSolder -> noggin:0805_LED_Extended
- moved VR1 1.78 mm to (131.3, 85.3)
Connections:
- VR1 pad 1: +5V -> +3V3
- VR1 pad 3: +3V3 -> +5V
Routing:
- net +3V3: track 315.6 -> 323.1 mm
- net +5V: track 30.4 -> 24.9 mm
